Commit message: third commit

File: urdf/tl1_1.urdf.xacro (robot description, xacro)
@@ -63,5 +63,6 @@
       <parent link="base_link"/>
       <child link="left_leg"/>
-      <origin xyz="0 ${(width/2+.06)} 0" rpy="0 ${pi/2} 0"/>
+      <!-- <origin xyz="0 ${(width/2+.06)} 0" rpy="0 ${pi/2} 0"/> -->
+      <origin xyz="0 ${(width/2+.06)} 0"/>
       <axis xyz="0 1 0"/>
       <limit effort="10" velocity="10"/>
@@ -91,5 +92,6 @@
       <parent link="base_link"/>
       <child link="right_leg"/>
-      <origin xyz="0 ${-1*(width/2+.06)} 0" rpy="0 ${pi/2} 0"/>
+      <!-- <origin xyz="0 ${-1*(width/2+.06)} 0" rpy="0 ${pi/2} 0"/> -->
+      <origin xyz="0 ${-1*(width/2+.06)} 0"/>
       <axis xyz="0 1 0"/>
       <limit effort="10" velocity="10"/>
